Commit message: ADD 添加了diffbot的中文注释;添加了rviz的部分教程; Change 四组轮滑机器人关节的坐标轴,仍有报错,不能运动

File: src/four_skating/urdf/four_skating.urdf (robot description, URDF)
Before this commit: robot four_skating, 13 links, 12 joints
Links:
- removed link left_backward_Link_1
- removed link left_backward_Link_2
- removed link left_backward_lun
- removed link left_forward_Link_1
- removed link left_forward_Link_2
- removed link left_forward_lun
- removed link right_backward_Link_1
- removed link right_backward_Link_2
- removed link right_backward_lun
- removed link right_forward_Link_1
- removed link right_forward_Link_2
- removed link right_forward_lun
- added link left_backward_link_1, mass 0.00155580902775302; collision mesh filename=package://four_skating/meshes/left_backward_link_1.STL; visual mesh filename=package://four_skating/meshes/left_backward_link_1.STL
- added link left_backward_link_2, mass 0.000410674770424681; collision mesh filename=package://four_skating/meshes/left_backward_link_2.STL; visual mesh filename=package://four_skating/meshes/left_backward_link_2.STL
- added link left_backward_wheel_link, mass 0.00235619449019234; collision mesh filename=package://four_skating/meshes/left_backward_wheel_link.STL; visual mesh filename=package://four_skating/meshes/left_backward_wheel_link.STL
- added link left_forward_link_1, mass 0.00155580902775302; collision mesh filename=package://four_skating/meshes/left_forward_link_1.STL; visual mesh filename=package://four_skating/meshes/left_forward_link_1.STL
- added link left_forward_link_2, mass 0.000410674770424681; collision mesh filename=package://four_skating/meshes/left_forward_link_2.STL; visual mesh filename=package://four_skating/meshes/left_forward_link_2.STL
- added link left_forward_wheel_link, mass 0.00235619449019234; collision mesh filename=package://four_skating/meshes/left_forward_wheel_link.STL; visual mesh filename=package://four_skating/meshes/left_forward_wheel_link.STL
- added link right_backward_link_1, mass 0.00155580902775302; collision mesh filename=package://four_skating/meshes/right_backward_link_1.STL; visual mesh filename=package://four_skating/meshes/right_backward_link_1.STL
- added link right_backward_link_2, mass 0.000410674770424681; collision mesh filename=package://four_skating/meshes/right_backward_link_2.STL; visual mesh filename=package://four_skating/meshes/right_backward_link_2.STL
- added link right_backward_wheel_link, mass 0.00235619449019235; collision mesh filename=package://four_skating/meshes/right_backward_wheel_link.STL; visual mesh filename=package://four_skating/meshes/right_backward_wheel_link.STL
- added link right_forward_link_1, mass 0.00155580902775302; collision mesh filename=package://four_skating/meshes/right_forward_link_1.STL; visual mesh filename=package://four_skating/meshes/right_forward_link_1.STL
- added link right_forward_link_2, mass 0.000410674770424681; collision mesh filename=package://four_skating/meshes/right_forward_link_2.STL; visual mesh filename=package://four_skating/meshes/right_forward_link_2.STL
- added link right_forward_wheel_link, mass 0.00235619449019235; collision mesh filename=package://four_skating/meshes/right_forward_wheel_link.STL; visual mesh filename=package://four_skating/meshes/right_forward_wheel_link.STL
Joints:
- removed joint left_backward_Joint_1
- removed joint left_backward_Joint_2
- removed joint left_backward_lun
- removed joint left_forward_Joint_1
- removed joint left_forward_Joint_2
- removed joint left_forward_lun
- removed joint right_backward_Joint_1
- removed joint right_backward_Joint_2
- removed joint right_backward_lun
- removed joint right_forward_Joint_1
- removed joint right_forward_Joint_2
- removed joint right_forward_lun
- added joint left_backward_joint_1: type continuous, parent base_link, child left_backward_link_1, origin xyz=-0.04 0.025 0 rpy=1.5708 0 -2.7407, axis 0 0 1
- added joint left_backward_joint_2: type prismatic, parent left_backward_link_1, child left_backward_link_2, origin xyz=0 0.005 0.00812196270704283 rpy=3.14159265358979 0 3.14159265358979, axis 0 0 1, limit lower=0 upper=0 effort=0 velocity=0
- added joint left_backward_wheel_joint: type continuous, parent left_backward_link_2, child left_backward_wheel_link, origin xyz=0 0 -0.0161637941803131 rpy=0 0 -0.206289656954149, axis 0 0 1
- added joint left_forward_joint_1: type continuous, parent base_link, child left_forward_link_1, origin xyz=0.0399999999999999 0.0250000000000002 0 rpy=1.5707963267949 0 3.02538154316369, axis 0 0 1
- added joint left_forward_joint_2: type prismatic, parent left_forward_link_1, child left_forward_link_2, origin xyz=0 0.005 0.019733 rpy=3.1416 0 3.1416, axis 0 0 1, limit lower=0 upper=0 effort=0 velocity=0
- added joint left_forward_wheel_joint: type continuous, parent left_forward_link_2, child left_forward_wheel_link, origin xyz=0 0 -0.0246638915913767 rpy=0 0 2.54006675826632, axis 0 0 1
- added joint right_backward_joint_1: type continuous, parent base_link, child right_backward_link_1, origin xyz=-0.04 -0.025 0 rpy=1.5707963267949 0 -0.264786446467445, axis 0 0 1
- added joint right_backward_joint_2: type prismatic, parent right_backward_link_1, child right_backward_link_2, origin xyz=0 0.00500000000000001 0.0181150724675244 rpy=-3.14159265358979 0 3.14159265358979, axis 0 0 1, limit lower=0 upper=0 effort=0 velocity=0
- added joint right_backward_wheel_joint: type continuous, parent right_backward_link_2, child right_backward_wheel_link, origin xyz=0 0 -0.0232877863584131 rpy=0 0 -0.377256984560737, axis 0 0 1
- added joint right_forward_joint_1: type continuous, parent base_link, child right_forward_link_1, origin xyz=0.04 -0.025 0 rpy=1.5708 0 0.50352, axis 0 0 1
- added joint right_forward_joint_2: type prismatic, parent right_forward_link_1, child right_forward_link_2, origin xyz=0 0.005 0.00583598115499422 rpy=-3.14159265358979 0 3.14159265358979, axis 0 0 1, limit lower=0 upper=0 effort=0 velocity=0
- added joint right_forward_wheel_joint: type continuous, parent right_forward_link_2, child right_forward_wheel_link, origin xyz=0 0 -0.0131949860626701 rpy=0 0 -1.15776168458666, axis 0 0 1
